File: project_v1/STM32_audio_KiCAD/STM32_audio.kicad_sch (KiCad schematic)
At the start: 79 parts, among them J1 Screw_Terminal_01x02, J2 SWD, J3 Conn_01x04, J4 Conn_01x04, J5 USB_B_Mini, J6 AudioJack3_Ground, J7 Micro_SD_Card_Det2, Q1 AO3401A, SW1 SW_SPDT, U1 STM32F405RGT6, U3 USBLC6-2SC6, U4 PCM5102A, Y1 16MHz

Commit message: Ajout Capteurs
update sch pour intégrer OLED, BP et module photoresistance
update documentation
Parts:
- added C30: C, Capacitor_SMD:C_0805_2012Metric, symbol Device:C
- added R27, R28: R, Resistor_SMD:R_0805_2012Metric, symbol Device:R
- added SW2: SW_Push, Button_Switch_SMD:SW_Push_1P1T_NO_CK_KSC6xxG, symbol Switch:SW_Push
Connections:
- net +3.3V: now also R28.1; no longer U1.64 (VDD)
- net GND: now also C30.2, SW2.1
- net PHOTOR_ADC: now reaches U1.8 (PC0)
- new net: R27.1, SW2.2
- new net ALARM_DIS: C30.1, R27.2, R28.2
- no-connect marks 33 -> 32
Other:
- added sheet Capteurs (capteurs.kicad_sch)
- note added: "Exemple boutton poussoir"
- note added: "Modèle à choisir + Footprint"
- moved on the sheet: D1, R3
