File: HW/STM32_audio_KiCAD/STM32_audio.kicad_sch (KiCad schematic)
At the start: 92 parts, among them J1 Conn_01x01_Socket, J10 Conn_01x01_Socket, J11 Conn_01x01_Socket, J12 Conn_01x01_Socket, J13 Conn_01x01_Socket, J2 SWD (Serial Wire Debug connec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, J3 Conn_01x01_Socket, J4 Conn_01x01_Socket, J5 USB_B_Mini, J6 AudioJack3_Ground, J7 Micro_SD_Card_Det2, J8 KY-018, J9 OLED_0,96", Q1 AO3401A, SW1 SW_SPDT, SW2 SW_Push, U1 STM32F405RGT6, U3 USBLC6-2SC6, U4 PCM5102A, U5 LP2985-3.3, Y1 16MHz

Commit message: Correction schéma
- Ajout d'un condensateur au bouton poussoir
- Ajout capteur de lumière
- Update de l'organisation générale du schematic
Parts:
- added C34: 1uF, OptoDevice:AMS_TSL25911FN, symbol Device:C_Small
- added C35: 100nF, symbol Device:C_Small
- added R16: 10k, Resistor_THT:R_Array_SIP4, symbol Device:R_Small
- added U6: TSL25911FN, OptoDevice:AMS_TSL25911FN, symbol Sensor_Optical:TSL25911FN
Connections:
- net +3.3V: now also C34.1, R16.2, U6.5 (VDD)
- net ALARM_DIS: now also U1.26 (PB0), C35.1
- net GND: now also C34.2, C35.2, U6.3 (GND)
- net I2C1_SCL: now also U6.1 (SCL)
- net I2C1_SDA: now also U6.6 (SDA)
- net PHOTOR_ADC: now also U1.8 (PC0)
- net EXTI1: now reaches U1.9 (PC1)
- net EXTI1: now also R16.1, U6.2 (INT)
- no-connect marks 32 -> 29
Other:
- note added: "Capteur de lumière TSL25911FN"
- note added: "Ecran OLED 0,96 pouce"
- moved on the sheet: D1, J10, J11, J3, J4, J9, R14, R15, R28, R3, SW2, U3
