File: HW/STM32_audio_KiCAD/STM32_audio.kicad_pcb (KiCad board)
At the start: 4 copper layers, 91.2 x 66.8 mm, 101 parts, among them J1 Conn_01x02_Socket, J10 Conn_01x01_Socket, J11 Conn_01x01_Socket, J12 Conn_01x01_Socket, J13 Conn_01x01_Socket, J15 Conn_01x06_Socket, J2 Conn_01x04_Socket, J3 Conn_01x01_Socket, J4 Conn_01x01_Socket, J5 USB_B_Mini, J6 AudioJack3_Ground, J7 Micro_SD_Card_Det2, J8 KY-018, J9 OLED_0,96", Q1 AO3401A, SW1 SW_SPDT, SW2 SW_Push, U1 STM32F405RGT6, U3 USBLC6-2SC6, U4 PCM5102A, U5 LP2985-3.3, U6 TSL25911FN, Y1 16MHz

Commit message: Update Footprint and Routing
- ERC correct
- Schematic à jour
- MX à jour
- Footprint checké
- Routing bien commencé
Routing:
- net GND: track 0.00 -> 257.5 mm, vias 0 -> 9
- net ADC_DVDD: track 0.00 -> 148.1 mm, vias 0 -> 7
- net SD_DET: track 0.00 -> 71.7 mm, vias 0 -> 2
- net ALARM_DISABLE: track 0.00 -> 65.0 mm
- net ADC_AVDD: track 0.00 -> 57.3 mm, vias 0 -> 2
- net ADC_AGND: track 0.00 -> 53.1 mm, vias 0 -> 2
- net SD_CLK: track 0.00 -> 42.5 mm, vias 0 -> 2
- net Net-(J2-Pin_2): track 0.00 -> 40.6 mm, vias 0 -> 2
- net SD_D0: track 0.00 -> 40.1 mm, vias 0 -> 4
- net ADC_DGND: track 0.00 -> 39.5 mm, vias 0 -> 2
- net SD_D1: track 0.00 -> 38.7 mm, vias 0 -> 6
- net I2C1_SCL: track 0.00 -> 30.5 mm, vias 0 -> 4
- net BUCK_IN: track 0.00 -> 29.5 mm, vias 0 -> 3
- net I2C1_SDA: track 0.00 -> 25.9 mm, vias 0 -> 5
- net SWDIO: track 0.00 -> 22.1 mm
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