File: HW/STM32_audio_KiCAD/STM32_audio.kicad_pcb (KiCad board)
At the start: 4 copper layers, 91.2 x 66.8 mm, 101 parts, among them J1 Conn_01x02_Socket, J10 Conn_01x01_Socket, J11 Conn_01x01_Socket, J12 Conn_01x01_Socket, J13 Conn_01x01_Socket, J15 Conn_01x06_Socket, J2 Conn_01x04_Socket, J3 Conn_01x01_Socket, J4 Conn_01x01_Socket, J5 USB_B_Mini, J6 AudioJack3_Ground, J7 Micro_SD_Card_Det2, J8 KY-018, J9 OLED_0,96", Q1 AO3401A, SW1 SW_SPDT, SW2 SW_Push, U1 STM32F405RGT6, U3 USBLC6-2SC6, U4 PCM5102A, U5 LP2985-3.3, U6 TSL25911FN, Y1 16MHz

Commit message: Save
Parts:
- removed J10, J11, J3, J4: Conn_01x01_Socket, Connector_PinSocket_2.54mm:PinSocket_1x01_P2.54mm_Vertical
- moved J15 212.3 mm to (181.0, 115.0), turned to -90 degrees
- moved C36 173.8 mm to (164.0, 70.5)
- moved C37 159.4 mm to (150.0, 68.5)
- moved C38 159.4 mm to (150.0, 70.5)
- moved R27 156.4 mm to (150.0, 65.0)
- moved H2 11.0 mm to (107.0, 111.2)
- moved J2 2.79 mm to (188.0, 54.5)
- moved SW1 1.06 mm to (158.0, 52.0), turned to 180 degrees
Routing:
- net GND: track 257.5 -> 309.2 mm, vias 9 -> 14
- net ADC_DGND: track 39.5 -> 1.87 mm, vias 2 -> 0
- net ADC_AVDD: track 57.3 -> 47.0 mm
- net ADC_AGND: track 53.1 -> 62.1 mm, vias 2 -> 3
- net ADC_DVDD: track 148.1 -> 144.9 mm
- net ADC_CAPM: track 1.13 -> 3.77 mm
Other:
- board size 91.2 x 66.8 mm -> 102.7 x 66.8 mm
